File: kicad/z80_nop.kicad_sch (KiCad schematic)
At the start: 32 parts, among them J1 USB_C_Receptacle_PowerOnly_6P, J2 USB_A, J3 USB_B_Micro, SW1 SW_Push, U1 NE555, U2 Z80CPU

Commit message: Minor tweaks
Parts:
- removed J3: USB_B_Micro, Connector_USB:USB_Micro-B_Amphenol_10103594-0001LF_Horizontal, symbol Connector:USB_B_Micro
- added J5: Barrel_Jack, Connector_BarrelJack:BarrelJack_Wuerth_6941xx301002, symbol Connector:Barrel_Jack
- added TP10: ~{M1}, TestPoint:TestPoint_THTPad_2.0x2.0mm_Drill1.0mm, symbol Connector:TestPoint
- added TP11: ~{RFSH}, TestPoint:TestPoint_THTPad_2.0x2.0mm_Drill1.0mm, symbol Connector:TestPoint
- added TP8: ~{RD}, TestPoint:TestPoint_THTPad_2.0x2.0mm_Drill1.0mm, symbol Connector:TestPoint
- added TP9: ~{MREQ}, TestPoint:TestPoint_THTPad_2.0x2.0mm_Drill1.0mm, symbol Connector:TestPoint
- RV1: value 1M -> 2M
- U1: value NE555 -> LM555CN
- U2: value Z80CPU -> Z80
Connections:
- net GND: now also J5.2
- net M1: now also TP10.1
- net MREQ: now also TP9.1
- net PWR: now also R3.2, J5.1
- net RD: now also TP8.1
- net RFSH: now also TP11.1
- net at R3.1, U2.26 (~{RESET}): now also SW1.1
- no-connect marks 7 -> 4
Other:
- note added: "1nf + 100nf -> 325Hz to 22KHz Approx 2.2nf + 47nF -> 150Hz to 10KHz Approx"
- note added: "Approx 250Hz to 20KHz"
- note added: "D6L90 F2 LFS"
- note added: "PT10LV10-205A2020-S"
- note added: "WURTH ELEKTRONIK 694108301002"
- note removed: "10103594-0001LF"
- note removed: "Approx 20 to 800Hz"
- moved on the sheet: SW1

Commit message: Update docs
Other:
- note added: "1nf -> 325Hz to 22KHz Approx 2.2nf -> 150Hz to 10KHz Approx 4.7nf -> 75Hz to 5KHz approx"
- note removed: "1nf + 100nf -> 325Hz to 22KHz Approx 2.2nf + 47nF -> 150Hz to 10KHz Approx"
Changed lines of the file:
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@@
 		)
 	)
-	(text "1nf + 100nf -> 325Hz to 22KHz Approx\n2.2nf + 47nF -> 150Hz to 10KHz Approx"
+	(text "1nf  -> 325Hz to 22KHz Approx\n2.2nf  -> 150Hz to 10KHz Approx\n4.7nf  -> 75Hz to 5KHz approx\n"
 		(exclude_from_sim no)
-		(at 99.822 123.698 0)
+		(at 49.276 100.838 0)
 		(effects
 			(font
@@
 				(thickness 0.1588)
 			)
+			(justify left)
 		)
 	)

Commit message: Add HALT mode
Parts:
- removed RN1: 4.7K, Resistor_THT:R_Array_SIP9, symbol Device:R_Network08
- added C4: 10nF, Capacitor_THT:C_Disc_D6.0mm_W2.5mm_P5.00mm, symbol Device:C
- added RN1: R_Pack08, Package_DIP:DIP-16_W7.62mm, symbol Device:R_Pack08
- added SW2: SW_SPDT, 80_Bus:SW_Slide-03_Pin-2-Common_10x2.5x6.4_P2.54mm, symbol Switch:SW_SPDT
- SW1: footprint 80_Bus:SW_PUSH_5mm_H5mm -> Button_Switch_THT:SW_PUSH_6mm_H5mm
- TP6: value ~{HALT} -> ~{RD}
- TP8: value ~{RD} -> ~{HALT}
Connections:
- net GND: now also RN1.1 (R1.1), RN1.5 (R5.1), RN1.8 (R8.1), SW2.1 (A)
- net M1: now also BAR2.2 (A); no longer BAR2.8 (A)
- net MREQ: now also BAR2.1 (A); no longer BAR2.9 (A)
- net PWR: now also SW2.3 (C)
- net RD: no longer BAR2.10 (A), TP8.1, U2.21 (~{RD})
- net RFSH: now also BAR2.3 (A); no longer BAR2.7 (A)
- net at BAR1.1 (A): now also U2.36 (A6); no longer U2.5 (A15)
- net at BAR1.10 (A): now also U2.5 (A15); no longer U2.36 (A6)
- net at BAR1.11 (K): now also RN2.9 (R8); no longer RN3.8 (R7)
- net at BAR1.12 (K): now also RN2.8 (R7); no longer RN3.9 (R8)
- net at BAR1.13 (K): now also RN2.7 (R6); no longer RN2.2 (R1)
- net at BAR1.14 (K): now also RN2.6 (R5); no longer RN2.3 (R2)
- net at BAR1.15 (K): now also RN2.5 (R4); no longer RN2.4 (R3)
- net at BAR1.16 (K): now also RN2.4 (R3); no longer RN2.5 (R4)
- net at BAR1.17 (K): now also RN2.3 (R2); no longer RN2.6 (R5)
- net at BAR1.18 (K): now also RN2.2 (R1); no longer RN2.7 (R6)
- net at BAR1.19 (K): now also RN3.9 (R8); no longer RN2.8 (R7)
- net at BAR1.2 (A): now also U2.37 (A7); no longer U2.4 (A14)
- net at BAR1.20 (K): now also RN3.8 (R7); no longer RN2.9 (R8)
- net at BAR1.3 (A): now also U2.38 (A8); no longer U2.3 (A13)
- net at BAR1.4 (A): now also U2.39 (A9); no longer U2.2 (A12)
- net at BAR1.5 (A): now also U2.40 (A10); no longer U2.1 (A11)
- net at BAR1.6 (A): now also U2.1 (A11); no longer U2.40 (A10)
- net at BAR1.7 (A): now also U2.2 (A12); no longer U2.39 (A9)
- net at BAR1.8 (A): now also U2.3 (A13); no longer U2.38 (A8)
- net at BAR1.9 (A): now also U2.4 (A14); no longer U2.37 (A7)
- net at U2.35 (A5): now also BAR2.10 (A); no longer BAR2.1 (A)
- net at BAR2.11 (K): now also RN3.7 (R6); no longer RN4.2 (R1)
- net at BAR2.12 (K): now also RN3.6 (R5); no longer RN4.3 (R2)
- net at BAR2.13 (K): now also RN3.5 (R4); no longer RN4.4 (R3)
- net at BAR2.14 (K): now also RN3.4 (R3); no longer RN4.5 (R4)
- net at BAR2.15 (K): now also RN3.3 (R2); no longer RN3.2 (R1)
- net at BAR2.16 (K): now also RN3.2 (R1); no longer RN3.3 (R2)
- net at BAR2.17 (K): now also RN4.5 (R4); no longer RN3.4 (R3)
- net at BAR2.18 (K): now also RN4.4 (R3); no longer RN3.5 (R4)
- net at BAR2.19 (K): now also RN4.3 (R2); no longer RN3.6 (R5)
- net at U2.34 (A4): now also BAR2.9 (A); no longer BAR2.2 (A)
- net at BAR2.20 (K): now also RN4.2 (R1); no longer RN3.7 (R6)
- net at U2.33 (A3): now also BAR2.8 (A); no longer BAR2.3 (A)
- net at U2.32 (A2): now also BAR2.7 (A); no longer BAR2.4 (A)
- net at BAR2.5 (A): now also U2.30 (A0); no longer U2.31 (A1)
- net at BAR2.6 (A): now also U2.31 (A1); no longer U2.30 (A0)
- net at U2.14 (D0): now also RN1.9 (R8.2)
- net at U2.15 (D1): now also RN1.10 (R7.2)
- net at U2.12 (D2): now also RN1.11 (R6.2)
- net at U2.8 (D3): now also RN1.12 (R5.2)
- net at U2.7 (D4): now also RN1.13 (R4.2)
- net at U2.9 (D5): now also RN1.14 (R3.2)
- net at U2.10 (D6): now also RN1.15 (R2.2)
- net at U2.13 (D7): now also RN1.16 (R1.2)
- net at R3.1, SW1.1, U2.26 (~{RESET}): now also C4.1
- net at TP6.1: now also U2.21 (~{RD}); no longer U2.18 (~{HALT})
- new net: RN1.2 (R2.1), RN1.3 (R3.1), RN1.4 (R4.1), RN1.6 (R6.1), RN1.7 (R7.1), SW2.2 (B)
- new net HALT: BAR2.4 (A), TP8.1, U2.18 (~{HALT})
Other:
- note added: "4116R-1-472"
- note added: "HALT Mode"
- note added: "NOP Mode"
- note added: "OSX10201-RGG"
- note removed: "4609M-101-472LF"
- note removed: "D6L90 F2 LFS"
- title: Z80 NOP TEster -> Z80 HALT NOP Tester
- moved on the sheet: BAR1, BAR2, H1, H2, H3, H4, TP6, TP7
